File: showcase/showcase.kicad_pcb (KiCad board)
At the start: 2 copper layers, 914.4 x 519.1 mm, 195 parts

Commit message: update showcase
Parts:
- added REF**: KEY_SWITCH, BrownSugar_KBD:Kailh_Choc_V2, F.Cu at (245.3, 488.2)
